File: mptt-controller.sch (EAGLE design)
At the start: 60 parts, among them IC1 ATSAMD09D14A-MU, Q1 MMBTA56LT1G, Q5 CSD18533KCS, Q6 CSD18533KCS, U1 AP2112K, U2 LM5109BMA/NOPB

Commit message: Very close to being finished.
Connections:
- net N$8 renamed VS
- new net N$3: IC1.PA09/I7/SERCOM1+0.3, R18.1
- net GND: now also JP1.8
- net P_EN: no longer IC1.PA09/I7/SERCOM1+0.3, R18.1
Changed lines of the file:
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@@
 <grid distance="0.1" unitdist="inch" unit="inch" style="lines" multiple="1" display="no" altdistance="0.01" altunitdist="inch" altunit="inch"/>
 <layers>
-<layer number="1" name="Top" color="4" fill="1" visible="yes" active="no"/>
-<layer number="16" name="Bottom" color="1" fill="1" visible="yes" active="no"/>
-<layer number="17" name="Pads" color="2" fill="1" visible="yes" active="no"/>
-<layer number="18" name="Vias" color="2" fill="1" visible="yes" active="no"/>
-<layer number="19" name="Unrouted" color="6" fill="1" visible="yes" active="no"/>
-<layer number="20" name="Dimension" color="24" fill="1" visible="yes" active="no"/>
-<layer number="21" name="tPlace" color="7" fill="1" visible="yes" active="no"/>
-<layer number="22" name="bPlace" color="7" fill="1" visible="yes" active="no"/>
-<layer number="23" name="tOrigins" color="15" fill="1" visible="yes" active="no"/>
-<layer number="24" name="bOrigins" color="15" fill="1" visible="yes" active="no"/>
-<layer number="25" name="tNames" color="7" fill="1" visible="yes" active="no"/>
-<layer number="26" name="bNames" color="7" fill="1" visible="yes" active="no"/>
-<layer number="27" name="tValues" color="7" fill="1" visible="yes" active="no"/>
-<layer number="28" name="bValues" color="7" fill="1" visible="yes" active="no"/>
+<layer number="1" name="Top" color="4" fill="1" visible="no" active="no"/>
+<layer number="16" name="Bottom" color="1" fill="1" visible="no" active="no"/>
+<layer number="17" name="Pads" color="2" fill="1" visible="no" active="no"/>
+<layer number="18" name="Vias" color="2" fill="1" visible="no" active="no"/>
+<layer number="19" name="Unrouted" color="6" fill="1" visible="no" active="no"/>
+<layer number="20" name="Dimension" color="24" fill="1" visible="no" active="no"/>
+<layer number="21" name="tPlace" color="7" fill="1" visible="no" active="no"/>
+<layer number="22" name="bPlace" color="7" fill="1" visible="no" active="no"/>
+<layer number="23" name="tOrigins" color="15" fill="1" visible="no" active="no"/>
+<layer number="24" name="bOrigins" color="15" fill="1" visible="no" active="no"/>
+<layer number="25" name="tNames" color="7" fill="1" visible="no" active="no"/>
+<layer number="26" name="bNames" color="7" fill="1" visible="no" active="no"/>
+<layer number="27" name="tValues" color="7" fill="1" visible="no" active="no"/>
+<layer number="28" name="bValues" color="7" fill="1" visible="no" active="no"/>
 <layer number="29" name="tStop" color="7" fill="3" visible="no" active="no"/>
 <layer number="30" name="bStop" color="7" fill="6" visible="no" active="no"/>
@@
 <layer number="35" name="tGlue" color="7" fill="4" visible="no" active="no"/>
 <layer number="36" name="bGlue" color="7" fill="5" visible="no" active="no"/>
-<layer number="37" name="tTest" color="7" fill="1" visible="yes" active="no"/>
-<layer number="38" name="bTest" color="7" fill="1" visible="yes" active="no"/>
+<layer number="37" name="tTest" color="7" fill="1" visible="no" active="no"/>
+<layer number="38" name="bTest" color="7" fill="1" visible="no" active="no"/>
 <layer number="39" name="tKeepout" color="4" fill="11" visible="no" active="no"/>
 <layer number="40" name="bKeepout" color="1" fill="11" visible="no" active="no"/>
@@
 <layer number="44" name="Drills" color="7" fill="1" visible="no" active="no"/>
 <layer number="45" name="Holes" color="7" fill="1" visible="no" active="no"/>
-<layer number="46" name="Milling" color="3" fill="1" visible="yes" active="no"/>
-<layer number="47" name="Measures" color="7" fill="1" visible="yes" active="no"/>
-<layer number="48" name="Document" color="7" fill="1" visible="yes" active="no"/>
-<layer number="49" name="Reference" color="7" fill="1" visible="yes" active="no"/>
-<layer number="50" name="dxf" color="7" fill="1" visible="yes" active="no"/>
-<layer number="51" name="tDocu" color="7" fill="1" visible="yes" active="no"/>
-<layer number="52" name="bDocu" color="7" fill="1" visible="yes" active="no"/>
-<layer number="53" name="tGND_GNDA" color="7" fill="9" visible="yes" active="no"/>
-<layer number="54" name="bGND_GNDA" color="1" fill="9" visible="yes" active="no"/>
-<layer number="56" name="wert" color="7" fill="1" visible="yes" active="no"/>
-<layer number="57" name="tCAD" color="7" fill="1" visible="yes" active="no"/>
-<layer number="59" name="tCarbon" color="7" fill="1" visible="yes" active="no"/>
-<layer number="60" name="bCarbon" color="7" fill="1" visible="yes" active="no"/>
+<layer number="46" name="Milling" color="3" fill="1" visible="no" active="no"/>
+<layer number="47" name="Measures" color="7" fill="1" visible="no" active="no"/>
+<layer number="48" name="Document" color="7" fill="1" visible="no" active="no"/>
+<layer number="49" name="Reference" color="7" fill="1" visible="no" active="no"/>
+<layer number="50" name="dxf" color="7" fill="1" visible="no" active="no"/>
+<layer number="51" name="tDocu" color="7" fill="1" visible="no" active="no"/>
+<layer number="52" name="bDocu" color="7" fill="1" visible="no" active="no"/>
+<layer number="53" name="tGND_GNDA" color="7" fill="9" visible="no" active="no"/>
+<layer number="54" name="bGND_GNDA" color="1" fill="9" visible="no" active="no"/>
+<layer number="56" name="wert" color="7" fill="1" visible="no" active="no"/>
+<layer number="57" name="tCAD" color="7" fill="1" visible="no" active="no"/>
+<layer number="59" name="tCarbon" color="7" fill="1" visible="no" active="no"/>
+<layer number="60" name="bCarbon" color="7" fill="1" visible="no" active="no"/>
 <layer number="88" name="SimResults" color="9" fill="1" visible="yes" active="yes"/>
 <layer number="89" name="SimProbes" color="9" fill="1" visible="yes" active="yes"/>
@@
 <instance part="R11" gate="G$1" x="243.84" y="144.78" smashed="yes" rot="R90">
 <attribute name="NAME" x="241.3" y="144.78" size="1.27" layer="95" font="vector" rot="R90" align="center"/>
-<attribute name="VALUE" x="243.84" y="144.78" size="1.016" layer="96" font="vector" ratio="15" rot="R90" align="center"/>
+<attribute name="VALUE" x="246.38" y="144.78" size="1.016" layer="96" font="vector" ratio="15" rot="R90" align="center"/>
 </instance>
 <instance part="R14" gate="G$1" x="236.22" y="139.7" smashed="yes" rot="R90">
@@
 <wire x1="-17.78" y1="248.92" x2="-25.4" y2="248.92" width="0.1524" layer="91"/>
 <label x="-25.4" y="248.92" size="1.27" layer="95" rot="R180" xref="yes"/>
+</segment>
+<segment>
+<pinref part="JP1" gate="A" pin="8"/>
+<wire x1="-22.86" y1="147.32" x2="-33.02" y2="147.32" width="0.1524" layer="91"/>
+<label x="-33.02" y="147.32" size="1.27" layer="95" rot="R180" xref="yes"/>
 </segment>
 </net>
@@
 </segment>
 <segment>
-<pinref part="IC1" gate="G$1" pin="PA09/I7/SERCOM1+0.3"/>
-<wire x1="269.24" y1="228.6" x2="284.48" y2="228.6" width="0.1524" layer="91"/>
-<pinref part="R18" gate="G$1" pin="1"/>
-</segment>
-<segment>
 <wire x1="294.64" y1="228.6" x2="297.18" y2="228.6" width="0.1524" layer="91"/>
 <label x="297.18" y="228.6" size="1.27" layer="95" xref="yes"/>
@@
 </segment>
 </net>
-<net name="N$8" class="0">
+<net name="VS" class="0">
 <segment>
 <pinref part="FB1" gate="G$1" pin="P$2"/>
@@
 </segment>
 </net>
+<net name="N$3" class="0">
+<segment>
+<pinref part="IC1" gate="G$1" pin="PA09/I7/SERCOM1+0.3"/>
+<pinref part="R18" gate="G$1" pin="1"/>
+<wire x1="269.24" y1="228.6" x2="284.48" y2="228.6" width="0.1524" layer="91"/>
+</segment>
+</net>

Commit message: Board documentation layer and add a cap for VREFA.
Parts:
- added C17: 0.1uF, ATSAMD09D14 Breakout rev B:CAP_CERAMIC_0402MP
- added JP2: (no value), Adafruit Metro M0 Express:HEADER-1X6ROUND
Connections:
- new net AREF: C17.1, IC1.PA03/I3/VREFA/AIN1, JP2.6
- new net PA10: IC1.PA10/I2/AI18/SERCOM0.2, JP1.3
- new net PA11: IC1.PA11/I3/AIN9/SERCOM0.3, JP1.4
- new net PA14: IC1.PA14/I2C/AIN6/SERCOM0.0, JP1.5
- new net PA15: IC1.PA15/I2C/I1/AIN7/SERCOM0.1, JP1.6
- new net PA16: IC1.PA16/I0/SERCOM1.2, JP1.7
- new net PA17: IC1.PA17/I1/SERCOM1.3, JP2.1
- new net PA22: IC1.PA22/I2C/I6/SERCOM1.0, JP2.2
- new net PA23: IC1.PA23/I2C/I7/SERCOM1.1, JP2.3
- new net PA24: IC1.PA24/I4/SERCOM1.2, JP2.4
- new net PA25: IC1.PA25/I5/SERCOM1.3, JP2.5
- net GND: now also C17.2
- net VCC_3V3: now also JP1.2
Changed lines of the file:
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@@
 <part name="C13" library="ATSAMD09D14 Breakout rev B" deviceset="CAP_CERAMIC" device="_0402MP" value="0.1uF"/>
 <part name="U$2" library="bourns" deviceset="PQ2614" device="" value="22uH PQ2614BHA-220K"/>
+<part name="JP2" library="Adafruit Metro M0 Express" deviceset="HEADER-1X6" device="ROUND"/>
+<part name="C17" library="ATSAMD09D14 Breakout rev B" deviceset="CAP_CERAMIC" device="_0402MP" value="0.1uF"/>
 </parts>
 <sheets>
@@
 <attribute name="VALUE" x="312.18" y="245.09" size="1.27" layer="96" font="vector" rot="R90" align="center"/>
 </instance>
+<instance part="JP2" gate="A" x="7.62" y="152.4" smashed="yes">
+<attribute name="NAME" x="1.27" y="163.195" size="1.778" layer="95"/>
+<attribute name="VALUE" x="1.27" y="142.24" size="1.778" layer="96"/>
+</instance>
+<instance part="C17" gate="G$1" x="307.34" y="228.6" smashed="yes">
+<attribute name="NAME" x="305.05" y="229.85" size="1.27" layer="95" font="vector" rot="R90" align="center"/>
+<attribute name="VALUE" x="309.64" y="229.85" size="1.27" layer="96" font="vector" rot="R90" align="center"/>
+</instance>
 </instances>
 <busses>
@@
 <wire x1="309.88" y1="220.98" x2="309.88" y2="193.04" width="0.1524" layer="91"/>
 <wire x1="279.4" y1="233.68" x2="279.4" y2="220.98" width="0.1524" layer="91"/>
-<wire x1="279.4" y1="220.98" x2="309.88" y2="220.98" width="0.1524" layer="91"/>
+<wire x1="279.4" y1="220.98" x2="307.34" y2="220.98" width="0.1524" layer="91"/>
 <junction x="309.88" y="220.98"/>
 <pinref part="C11" gate="G$1" pin="2"/>
+<wire x1="307.34" y1="220.98" x2="309.88" y2="220.98" width="0.1524" layer="91"/>
 <wire x1="274.32" y1="236.22" x2="274.32" y2="233.68" width="0.1524" layer="91"/>
 <wire x1="274.32" y1="233.68" x2="279.4" y2="233.68" width="0.1524" layer="91"/>
 <junction x="279.4" y="233.68"/>
+<pinref part="C17" gate="G$1" pin="2"/>
+<wire x1="307.34" y1="226.06" x2="307.34" y2="220.98" width="0.1524" layer="91"/>
+<junction x="307.34" y="220.98"/>
 </segment>
 <segment>
@@
 <pinref part="FB1" gate="G$1" pin="P$1"/>
 </segment>
+<segment>
+<pinref part="JP1" gate="A" pin="2"/>
+<wire x1="-22.86" y1="162.56" x2="-33.02" y2="162.56" width="0.1524" layer="91"/>
+<label x="-33.02" y="162.56" size="1.27" layer="95" rot="R180" xref="yes"/>
+</segment>
 </net>
 <net name="SWCLK" class="0">
@@
 </segment>
 </net>
+<net name="PA10" class="0">
+<segment>
+<pinref part="IC1" gate="G$1" pin="PA10/I2/AI18/SERCOM0.2"/>
+<wire x1="269.24" y1="226.06" x2="271.78" y2="226.06" width="0.1524" layer="91"/>
+<label x="271.78" y="226.06" size="1.27" layer="95" xref="yes"/>
+</segment>
+<segment>
+<pinref part="JP1" gate="A" pin="3"/>
+<wire x1="-22.86" y1="160.02" x2="-33.02" y2="160.02" width="0.1524" layer="91"/>
+<label x="-33.02" y="160.02" size="1.27" layer="95" rot="R180" xref="yes"/>
+</segment>
+</net>
+<net name="PA11" class="0">
+<segment>
+<pinref part="IC1" gate="G$1" pin="PA11/I3/AIN9/SERCOM0.3"/>
+<wire x1="269.24" y1="223.52" x2="271.78" y2="223.52" width="0.1524" layer="91"/>
+<label x="271.78" y="223.52" size="1.27" layer="95" xref="yes"/>
+</segment>
+<segment>
+<pinref part="JP1" gate="A" pin="4"/>
+<wire x1="-22.86" y1="157.48" x2="-33.02" y2="157.48" width="0.1524" layer="91"/>
+<label x="-33.02" y="157.48" size="1.27" layer="95" rot="R180" xref="yes"/>
+</segment>
+</net>
+<net name="PA14" class="0">
+<segment>
+<pinref part="IC1" gate="G$1" pin="PA14/I2C/AIN6/SERCOM0.0"/>
+<wire x1="269.24" y1="218.44" x2="271.78" y2="218.44" width="0.1524" layer="91"/>
+<label x="271.78" y="218.44" size="1.27" layer="95" xref="yes"/>
+</segment>
+<segment>
+<pinref part="JP1" gate="A" pin="5"/>
+<wire x1="-22.86" y1="154.94" x2="-33.02" y2="154.94" width="0.1524" layer="91"/>
+<label x="-33.02" y="154.94" size="1.27" layer="95" rot="R180" xref="yes"/>
+</segment>
+</net>
+<net name="PA15" class="0">
+<segment>
+<pinref part="IC1" gate="G$1" pin="PA15/I2C/I1/AIN7/SERCOM0.1"/>
+<wire x1="269.24" y1="215.9" x2="271.78" y2="215.9" width="0.1524" layer="91"/>
+<label x="271.78" y="215.9" size="1.27" layer="95" xref="yes"/>
+</segment>
+<segment>
+<pinref part="JP1" gate="A" pin="6"/>
+<wire x1="-22.86" y1="152.4" x2="-33.02" y2="152.4" width="0.1524" layer="91"/>
+<label x="-33.02" y="152.4" size="1.27" layer="95" rot="R180" xref="yes"/>
+</segment>
+</net>
+<net name="PA16" class="0">
+<segment>
+<pinref part="IC1" gate="G$1" pin="PA16/I0/SERCOM1.2"/>
+<wire x1="269.24" y1="213.36" x2="271.78" y2="213.36" width="0.1524" layer="91"/>
+<label x="271.78" y="213.36" size="1.27" layer="95" xref="yes"/>
+</segment>
+<segment>
+<pinref part="JP1" gate="A" pin="7"/>
+<wire x1="-22.86" y1="149.86" x2="-33.02" y2="149.86" width="0.1524" layer="91"/>
+<label x="-33.02" y="149.86" size="1.27" layer="95" rot="R180" xref="yes"/>
+</segment>
+</net>
+<net name="PA17" class="0">
+<segment>
+<pinref part="IC1" gate="G$1" pin="PA17/I1/SERCOM1.3"/>
+<wire x1="269.24" y1="210.82" x2="271.78" y2="210.82" width="0.1524" layer="91"/>
+<label x="271.78" y="210.82" size="1.27" layer="95" xref="yes"/>
+</segment>
+<segment>
+<pinref part="JP2" gate="A" pin="1"/>
+<wire x1="5.08" y1="160.02" x2="-2.54" y2="160.02" width="0.1524" layer="91"/>
+<label x="-2.54" y="160.02" size="1.27" layer="95" rot="R180" xref="yes"/>
+</segment>
+</net>
+<net name="PA22" class="0">
+<segment>
+<pinref part="IC1" gate="G$1" pin="PA22/I2C/I6/SERCOM1.0"/>
+<wire x1="269.24" y1="205.74" x2="271.78" y2="205.74" width="0.1524" layer="91"/>
+<label x="271.78" y="205.74" size="1.27" layer="95" xref="yes"/>
+</segment>
+<segment>
+<pinref part="JP2" gate="A" pin="2"/>
+<wire x1="5.08" y1="157.48" x2="-2.54" y2="157.48" width="0.1524" layer="91"/>
+<label x="-2.54" y="157.48" size="1.27" layer="95" rot="R180" xref="yes"/>
+</segment>
+</net>
+<net name="PA23" class="0">
+<segment>
+<pinref part="IC1" gate="G$1" pin="PA23/I2C/I7/SERCOM1.1"/>
+<wire x1="269.24" y1="203.2" x2="271.78" y2="203.2" width="0.1524" layer="91"/>
+<label x="271.78" y="203.2" size="1.27" layer="95" xref="yes"/>
+</segment>
+<segment>
+<pinref part="JP2" gate="A" pin="3"/>
+<wire x1="5.08" y1="154.94" x2="-2.54" y2="154.94" width="0.1524" layer="91"/>
+<label x="-2.54" y="154.94" size="1.27" layer="95" rot="R180" xref="yes"/>
+</segment>
+</net>
+<net name="PA24" class="0">
+<segment>
+<pinref part="IC1" gate="G$1" pin="PA24/I4/SERCOM1.2"/>
+<wire x1="269.24" y1="200.66" x2="271.78" y2="200.66" width="0.1524" layer="91"/>
+<label x="271.78" y="200.66" size="1.27" layer="95" xref="yes"/>
+</segment>
+<segment>
+<pinref part="JP2" gate="A" pin="4"/>
+<wire x1="5.08" y1="152.4" x2="-2.54" y2="152.4" width="0.1524" layer="91"/>
+<label x="-2.54" y="152.4" size="1.27" layer="95" rot="R180" xref="yes"/>
+</segment>
+</net>
+<net name="PA25" class="0">
+<segment>
+<pinref part="IC1" gate="G$1" pin="PA25/I5/SERCOM1.3"/>
+<wire x1="271.78" y1="198.12" x2="269.24" y2="198.12" width="0.1524" layer="91"/>
+<label x="271.78" y="198.12" size="1.27" layer="95" xref="yes"/>
+</segment>
+<segment>
+<pinref part="JP2" gate="A" pin="5"/>
+<wire x1="5.08" y1="149.86" x2="-2.54" y2="149.86" width="0.1524" layer="91"/>
+<label x="-2.54" y="149.86" size="1.27" layer="95" rot="R180" xref="yes"/>
+</segment>
+</net>
+<net name="AREF" class="0">
+<segment>
+<pinref part="IC1" gate="G$1" pin="PA03/I3/VREFA/AIN1"/>
+<wire x1="269.24" y1="246.38" x2="307.34" y2="246.38" width="0.1524" layer="91"/>
+<pinref part="C17" gate="G$1" pin="1"/>
+<wire x1="307.34" y1="246.38" x2="307.34" y2="233.68" width="0.1524" layer="91"/>
+<wire x1="307.34" y1="246.38" x2="320.04" y2="246.38" width="0.1524" layer="91"/>
+<junction x="307.34" y="246.38"/>
+<label x="320.04" y="246.38" size="1.27" layer="95" xref="yes"/>
+</segment>
+<segment>
+<pinref part="JP2" gate="A" pin="6"/>
+<wire x1="5.08" y1="147.32" x2="-2.54" y2="147.32" width="0.1524" layer="91"/>
+<label x="-2.54" y="147.32" size="1.27" layer="95" rot="R180" xref="yes"/>
+</segment>
+</net>
